Commit message: Robot Now is Loaded Into the Scene

File: LiDAR_Simulation/heatsim_ws/src/ember_robot/model/robot.xacro (robot description, xacro)
@@ -5,12 +5,11 @@
 <!-- URDF DESCRIPTION OF THE DIFFERENTIAL DRIVE ROBOT    -->
 <!-- Reference/Source Aleksandar Haber                   -->
-<!-- Refer to liscence for questions                     -->
-<!-- ################################################    -->
-<robot name="ember_bot" xmlns:xacro="https://www.ros.org/wiki/xacro">
+<!-- Refer to licence for questions                      -->
+<!-- ################################################    -->
+<robot name="ember_bot" xmlns:xacro="http://www.ros.org/wiki/xacro">
 <!-- ################################################    -->
 <!--            Geometry & Constants                     -->
 <!--            MARK: G & C                              -->
 <!-- ################################################    -->
-<!-- Pi Constant-->
 <xacro:property name="pi_const" value="3.14159265"/>
 <!-- Body Dimensions -->
@@ -19,83 +18,64 @@
 <xacro:property name="c" value="0.6"/>
 <!-- Wheel & Caster Dimensions -->
-<!-- Wheel & Caser Radius -->
-<xacro:property name="r" value="0.15"/>
-<!-- Wheel Width -->
-<xacro:property name="d" value="0.1"/>
-<!-- Distances Between Certain Centres In Reference Robot -->
-<xacro:property name="s1" value="${b/2+r}"/>
-<xacro:property name="s2" value="${2*r}"/>
-<xacro:property name="s3" value="${2*r}"/>
-<xacro:property name="s4" value="${c/2+d/2}"/>
-<!-- ################################################    -->
+<xacro:property name="r" value="0.15"/> <!-- Radius -->
+<xacro:property name="d" value="0.1"/>  <!-- Width -->
+<!-- Distances Between Certain Centres -->
+<xacro:property name="s1" value="${b/2 + r}"/>
+<xacro:property name="s2" value="${r*2}"/>
+<xacro:property name="s3" value="${r*2}"/>
+<xacro:property name="s4" value="${c/2 + d/2}"/>
 <!-- ################################################    -->
 <!--                  Mass & Inertia                     -->
 <!--                  MARK: M & I                        -->
 <!-- ################################################    -->
-<!-- Material Density -->
-<!-- Body <Material Density> -->
-<xacro:property name="d1" value="2710.0"/>
-<!-- Wheel <Material Density> -->
-<xacro:property name="d2" value="2710.0"/>
-<!-- Caster <Material Density> -->
-<xacro:property name="d3" value="2710.0"/>
-<!-- Robot Body, Wheel, and Caster Mass -->
-<!-- Body <Mass> -->
+<!-- Densities -->
+<xacro:property name="d1" value="2710.0"/>  <!-- body -->
+<xacro:property name="d2" value="2710.0"/>  <!-- wheel -->
+<xacro:property name="d3" value="2710.0"/>  <!-- caster -->
+<!-- Masses -->
 <xacro:property name="m1" value="${d1*a*b*c}"/>
-<!-- Wheel <Mass> -->
 <xacro:property name="m2" value="${d2*pi_const*r*r*d}"/>
-<!-- Caster <Mass> -->
 <xacro:property name="m3" value="${d3*(4.0/3.0)*pi_const*r*r*r}"/>
-<!-- Moments of Inertia of the Robot Body -->
-<!-- Note Due to reference bot being symmetric, number of inertias are cut in half -->
-<xacro:property name="Ix_body" value="${(1/12)*m1*(b*b+c*c)}"/>
-<xacro:property name="Iy_body" value="${(1/12)*m1*(a*a+b*b)}"/>
-<xacro:property name="Iz_body" value="${(1/12)*m1*(a*a+c*c)}"/>
-<!-- Moments of Intertia of the Wheel -->
+<!-- Body inertia -->
+<xacro:property name="Ix_body" value="${(1.0/12.0)*m1*(b*b + c*c)}"/>
+<xacro:property name="Iy_body" value="${(1.0/12.0)*m1*(a*a + b*b)}"/>
+<xacro:property name="Iz_body" value="${(1.0/12.0)*m1*(a*a + c*c)}"/>
+<!-- Wheel inertia -->
 <xacro:property name="Iz_wheel" value="${0.5*m2*r*r}"/>
-<xacro:property name="I_wheel" value="${(1.0/12.0)*m2*(3.0*r*r+d*d))}"/>
-<!-- Moments of Inertia of the Caster Sphere -->
-<xacro:property name="I_caster" value="${(2.0/5.0)*m3*r*r)}"/>
-<!-- This Macro Defines the Complete Inertial Section of the Robot Body -->
-<!-- Utilized Later in the Code -->
+<xacro:property name="I_wheel" value="${(1.0/12.0)*m2*(3.0*r*r + d*d)}"/>
+<!-- Caster inertia -->
+<xacro:property name="I_caster" value="${(2.0/5.0)*m3*r*r}"/>
+<!-- Inertia macros -->
 <xacro:macro name="inertia_body">
     <inertial>
         <mass value="${m1}"/>
-        <inertia ixx="${Ix_body}" ixy="0.0" ixz="0.0" iyy="${Iy_body}" iyz="0" izz="${Iz_body}"/>
+        <inertia ixx="${Ix_body}" ixy="0" ixz="0" iyy="${Iy_body}" iyz="0" izz="${Iz_body}"/>
     </inertial>
 </xacro:macro>
-<!-- This Macro Defines the Complete Inertial Section of the Wheel -->
 <xacro:macro name="inertia_wheel">
     <inertial>
         <origin rpy="1.570795 0 0" xyz="0 0 0"/>
         <mass value="${m2}"/>
-        <inertia ixx="${I_wheel}" ixy="0.0" ixz="0.0" iyy="${I_wheel}" iyz="0" izz="${Iz_wheel}"/>
+        <inertia ixx="${I_wheel}" ixy="0" ixz="0" iyy="${I_wheel}" iyz="0" izz="${Iz_wheel}"/>
     </inertial>
 </xacro:macro>
-<!-- This Macro Defines the Complete Inertial Section of the Caster -->
 <xacro:macro name="inertia_caster">
     <inertial>
-        <origin rpy="0 0 0" xyz="0 0 0"/>
         <mass value="${m3}"/>
-        <inertia ixx="${I_caster}" ixy="0.0" ixz="0.0" iyy="${I_caster}" iyz="0" izz="${I_caster}"/>
+        <inertia ixx="${I_caster}" ixy="0" ixz="0" iyy="${I_caster}" iyz="0" izz="${I_caster}"/>
     </inertial>
 </xacro:macro>
-<!-- ################################################ -->
 <!-- ################################################ -->
 <!--            Include Additional Files              -->
 <!--            MARK: File Incl.                      -->
 <!-- ################################################ -->
-<!-- Over Here We Include the File that Defines Extra GZ Options and Motion Control Driver -->
 <xacro:include filename="$(find ember_robot)/model/robot.gazebo"/>
 <!-- ################################################ -->
-<!-- ################################################ -->
 <!-- MARK: LINKS, JOINTS HERE                        -->
 <!-- ################################################ -->
 <!-- ################################################ -->
-<!-- START: Fictious Link of the Robot                -->
-<!-- ################################################ -->
-<!-- Minute 26:07 of tutorial -->
-<!-- We need to have this link otherwise GZ will complain -->
-<link name="base_footprint"></link>
+<!-- START: Fictitious Link of the Robot              -->
+<!-- ################################################ -->
+<link name="base_footprint"/>
 <joint name="body_link_joint" type="fixed">
     <parent link="base_footprint"/>
@@ -103,5 +83,5 @@
 </joint>
 <!-- ################################################ -->
-<!-- END: Fictious Link of the Robot                  -->
+<!-- END: Fictitious Link of the Robot                -->
 <!-- ################################################ -->
 <!-- ################################################ -->
@@ -110,81 +90,70 @@
 <link name="body_link">
     <visual>
-        <geometry>
-            <box size="${a} ${c} ${b}"/>
-        </geometry>
-        <!-- Discplacement & Orientation of the Geomtric Centre of the link with respec to the link -->
-        <origin rpy="0 0 0" xyz="0 0 ${s1}"/>
-    </visual>
-    <!-- This allows for collision physics etc -->
-    <collision>
         <geometry>
             <box size="${a} ${c} ${b}"/>
         </geometry>
         <origin rpy="0 0 0" xyz="0 0 ${s1}"/>
+    </visual>
+    <collision>
+        <geometry>
+            <box size="${a} ${c} ${b}"/>
+        </geometry>
+        <origin rpy="0 0 0" xyz="0 0 ${s1}"/>
     </collision>
     <xacro:inertia_body/>
 </link>
 <!-- ################################################ -->
-<!-- End: Body Link of the Robot                      -->
-<!-- ################################################ -->
-<!-- ################################################  -->
-<!-- START: Back Right Wheel of the Robot and the Joint-->
-<!-- ################################################  -->
-<joint name="wheel_joint" type="continuous">
+<!-- END: Body Link of the Robot                      -->
+<!-- ################################################ -->
+<!-- ################################################  -->
+<!-- START: Back Right Wheel of the Robot + Joint      -->
+<!-- ################################################  -->
+<joint name="wheel1_joint" type="continuous">
     <parent link="body_link"/>
     <child link="wheel1_link"/>
     <origin xyz="${-s2} ${-s4} ${r}" rpy="0 0 0"/>
     <axis xyz="0 1 0"/>
-    <limit effort="50000" velocity="10"/>
-    <dynamics damping="1.0" friction="1.0"/>
 </joint>
 <link name="wheel1_link">
     <visual>
         <origin xyz="0 0 0" rpy="1.570795 0 0"/>
-        <geometry>
-            <cylinder radius="${r}" length="${d}"/>
-        </geometry>
-    </visual>
-    <collision>
-        <origin xyz="0 0 0" rpy="1.570795 0 0"/>
-        <geometry>
-            <cylinder radius="${r}" length="${d}"/>
-        </geometry>
+        <geometry><cylinder radius="${r}" length="${d}"/></geometry>
+    </visual>
+    <collision>
+        <origin xyz="0 0 0" rpy="1.570795 0 0"/>
+        <geometry><cylinder radius="${r}" length="${d}"/></geometry>
     </collision>
     <xacro:inertia_wheel/>
 </link>
 <!-- ################################################  -->
-<!-- END: Back Right Wheel of the Robot and the Joint  -->
-<!-- ################################################  -->
-<!-- ################################################  -->
-<!-- START: Back Left Wheel of the Robot and the Joint-->
-<!-- ################################################  -->
-<joint name="wheel_joint" type="continuous">
+<!-- END: Back Right Wheel                             -->
+<!-- ################################################  -->
+<!-- ################################################  -->
+<!-- START: Back Left Wheel of the Robot + Joint       -->
+<!-- ################################################  -->
+<joint name="wheel2_joint" type="continuous">
     <parent link="body_link"/>
     <child link="wheel2_link"/>
-    <origin xyz="${-s2} ${-s4} ${r}" rpy="0 0 0"/>
+    <origin xyz="${-s2} ${s4} ${r}" rpy="0 0 0"/>
     <axis xyz="0 1 0"/>
-    <limit effort="50000" velocity="10"/>
-    <dynamics damping="1.0" friction="1.0"/>
 </joint>
 <link name="wheel2_link">
     <visual>
         <origin xyz="0 0 0" rpy="1.570795 0 0"/>
-        <geometry>
-            <cylinder radius="${r}" length="${d}"/>
-        </geometry>
-    </visual>
-    <collision>
-        <origin xyz="0 0 0" rpy="1.570795 0 0"/>
-        <geometry>
-            <cylinder radius="${r}" length="${d}"/>
-        </geometry>
+        <geometry><cylinder radius="${r}" length="${d}"/></geometry>
+    </visual>
+    <collision>
+        <origin xyz="0 0 0" rpy="1.570795 0 0"/>
+        <geometry><cylinder radius="${r}" length="${d}"/></geometry>
     </collision>
     <xacro:inertia_wheel/>
 </link>
 <!-- ################################################  -->
-<!-- START: Caster Wheel                               -->
-<!-- ################################################  -->
-<joint name="caster_wheel" type="fixed">
+<!-- END: Back Left Wheel                              -->
+<!-- ################################################  -->
+<!-- ################################################  -->
+<!-- START: Caster Wheel                                -->
+<!-- ################################################  -->
+<joint name="caster_joint" type="fixed">
     <parent link="body_link"/>
     <child link="caster_link"/>
@@ -193,50 +162,39 @@
 <link name="caster_link">
     <visual>
-        <origin xyz="0 0 0" rpy="0 0 0"/>
-        <geometry>
-            <sphere radius="${r}"/>
-        </geometry>
-    </visual>
-    <collision>
-        <origin xyz="0 0 0" rpy="0 0 0"/>
-        <geometry>
-            <sphere radius="${r}"/>
-        </geometry>
+        <geometry><sphere radius="${r}"/></geometry>
+    </visual>
+    <collision>
+        <geometry><sphere radius="${r}"/></geometry>
     </collision>
     <xacro:inertia_caster/>
 </link>
 <!-- ################################################  -->
-<!-- END: Caster Wheel                                 -->
-<!-- ################################################  -->
-<!-- ################################################  -->
-<!-- START: LiDAR                                      -->
+<!-- END: Caster Wheel                                  -->
+<!-- ################################################  -->
+<!-- ################################################  -->
+<!-- START: LiDAR                                       -->
 <!-- ################################################  -->
 <joint name="lidar_joint" type="fixed">
-    <origin xyz="0.0 0 ${b+r}" rpy="0 0 0"/>
     <parent link="body_link"/>
     <child link="lidar_link"/>
-    <!--This means LiDAR should rotate around the y-axis -->
-    <origin xyz="0 1 0" rpy="0 0 0"/>
+    <origin xyz="0.0 0 0" rpy="0 0 0"/>
 </joint>
 <link name="lidar_link">
     <visual>
         <origin xyz="0 0 0.5" rpy="0 0 0"/>
-        <geometry>
-            <cylinder radius="0.1" length="0.1"/>
-        </geometry>
-    </visual>
-    <collision name="collision">
+        <geometry><cylinder radius="0.1" length="0.1"/></geometry>
+    </visual>
+    <collision>
         <origin xyz="0 0 0.5" rpy="0 0 0"/>
-        <geometry>
-            <cylinder radius="0.1" length="0.1"/>
-        </geometry>
-    </collision>
-    <inertial>
-        <mass value="le-6"/>
-    </inertial>
-    <xacro:inertia_caster/>
-</link>
-<!-- ################################################  -->
-<!-- END: LiDAR                                        -->
+        <geometry><cylinder radius="0.1" length="0.1"/></geometry>
+    </collision>
+    <!-- Minimal but valid inertia -->
+    <inertial>
+        <mass value="1e-6"/>
+        <inertia ixx="1e-6" ixy="0" ixz="0" iyy="1e-6" iyz="0" izz="1e-6"/>
+    </inertial>
+</link>
+<!-- ################################################  -->
+<!-- END: LiDAR                                         -->
 <!-- ################################################  -->
 </robot>

Commit message: Can Now Run Simulation and See LiDAR

File: LiDAR_Simulation/heatsim_ws/src/ember_robot/model/robot.xacro (robot description, xacro)
@@ -178,13 +178,13 @@
     <parent link="body_link"/>
     <child link="lidar_link"/>
-    <origin xyz="0.0 0 0" rpy="0 0 0"/>
+    <origin xyz="0.0 0 0.5" rpy="0 0 0"/>
 </joint>
 <link name="lidar_link">
     <visual>
-        <origin xyz="0 0 0.5" rpy="0 0 0"/>
+        <origin xyz="0 0 0" rpy="0 0 0"/>
         <geometry><cylinder radius="0.1" length="0.1"/></geometry>
     </visual>
     <collision>
-        <origin xyz="0 0 0.5" rpy="0 0 0"/>
+        <origin xyz="0 0 0" rpy="0 0 0"/>
         <geometry><cylinder radius="0.1" length="0.1"/></geometry>
     </collision>
