Commit message: ember.xacro added and md

File: LiDAR_Simulation/heatsim_ws/src/ember_robot/model/ember.xacro (robot description, xacro)
@@ -8,4 +8,5 @@
     attatched to the front, this LiDAR can be used in both
     2D and 3D modes.
+    *Note xacros are always in SI*
 -->
 <!-- ################################################    -->
@@ -39,4 +40,21 @@
 <!--            MARK: G & C                              -->
 <!-- ################################################    -->
+<!-- Track Dimensions -->
+<xacro:property name="tw" value="0.1"/>   <!-- Track width -->
+<xacro:property name="th" value="0.05"/>  <!-- Track height -->
+<xacro:property name="tl" value="0.3"/>   <!-- Track length -->
+<!-- Body Dimensions -->
+<xacro:property name="bw" value="0.3"/>  <!-- Body width -->
+<xacro:property name="bh" value="0.1"/>  <!-- Body height -->
+<xacro:property name="bl" value="0.3"/>  <!-- Body length -->
+<!-- LiDAR Dimensions -->
+<xacro:property name="lr" value="0.15"/> <!-- LiDAR Radius -->
+<xacro:property name="ll" value="0.1"/>  <!-- LiDAR Length -->
+<!-- TODO: Set Distances -->
+<!-- Distances Between Certain Centres -->
+<xacro:property name="s1" value="${b/2 + r}"/>
+<xacro:property name="s2" value="${r*2}"/>
+<xacro:property name="s3" value="${r*2}"/>
+<xacro:property name="s4" value="${c/2 + d/2}"/>
 <!-- ################################################    -->
 <!--                  Mass & Inertia                     -->
@@ -44,4 +62,9 @@
 <!-- ################################################    -->
 <!-- Densities -->
+<xacro:property name="body_desnity" value="2710.0"/>  <!-- body -->
+<xacro:property name="track_desnity" value="2710.0"/>  <!-- track -->
+ <!-- LiDAR density is not set as it would affect the spin of
+ the LiDAR if we were to set it. That being said the spin is
+ not simulated so we do not need to worry about it.-->
 <!-- Masses -->
 <!-- Body inertia -->

Commit message: 3d robot space beginnings

File: LiDAR_Simulation/heatsim_ws/src/ember_robot/model/ember.xacro (robot description, xacro)
@@ -63,5 +63,5 @@
 <!-- Densities -->
 <xacro:property name="body_desnity" value="2710.0"/>  <!-- body -->
-<xacro:property name="track_desnity" value="2710.0"/>  <!-- track -->
+<xacro:property name="track_desnity" value="2710.0"/>  <!-- track -->\
  <!-- LiDAR density is not set as it would affect the spin of
  the LiDAR if we were to set it. That being said the spin is

Commit message: added basic inertias

File: LiDAR_Simulation/heatsim_ws/src/ember_robot/model/ember.xacro (robot description, xacro)
@@ -68,6 +68,14 @@
  not simulated so we do not need to worry about it.-->
 <!-- Masses -->
+<xacro:property name="body_mass" value="${body_desnity*bl*bh*bw}"/>
+<xacro:property name="track_mass" value="${track_desnity*tl*th*tw}"/>
 <!-- Body inertia -->
+<xacro:property name="Ix_body" value="${(1.0/12.0)*body_mass*(bh*bh + bw*bw)}"/>
+<xacro:property name="Iy_body" value="${(1.0/12.0)*body_mass*(bl*bl + bh*bh)}"/>
+<xacro:property name="Iz_body" value="${(1.0/12.0)*body_mass*(bl*bl + bw*bw)}"/>
 <!-- Track inertia -->
+<xacro:property name="Ix_track" value="${(1.0/12.0)*mT*(tw*tw + th*th)}"/>
+<xacro:property name="Iy_track" value="${(1.0/12.0)*mT*(tl*tl + th*th)}"/>
+<xacro:property name="Iz_track" value="${(1.0/12.0)*mT*(tl*tl + tw*tw)}"/>
 <!-- Inertia macros -->
 <!-- ################################################ -->

Commit message: implemented basic distance setting

File: LiDAR_Simulation/heatsim_ws/src/ember_robot/model/ember.xacro (robot description, xacro)
@@ -34,6 +34,5 @@
  -->
 <!-- ################################################    -->
-<!-- TODO: When completed -->
-<!-- <robot name="ember_bot" xmlns:xacro="http://www.ros.org/wiki/xacro"> -->
+<robot name="ember_bot" xmlns:xacro="http://www.ros.org/wiki/xacro">
 <!-- ################################################    -->
 <!--            Geometry & Constants                     -->
@@ -41,20 +40,31 @@
 <!-- ################################################    -->
 <!-- Track Dimensions -->
-<xacro:property name="tw" value="0.1"/>   <!-- Track width -->
-<xacro:property name="th" value="0.05"/>  <!-- Track height -->
-<xacro:property name="tl" value="0.3"/>   <!-- Track length -->
+<xacro:property name="tl" value="0.30"/>   <!-- track length (X) -->
+<xacro:property name="tw" value="0.10"/>   <!-- track width  (Y) -->
+<xacro:property name="th" value="0.05"/>   <!-- track height (Z) -->
 <!-- Body Dimensions -->
-<xacro:property name="bw" value="0.3"/>  <!-- Body width -->
-<xacro:property name="bh" value="0.1"/>  <!-- Body height -->
-<xacro:property name="bl" value="0.3"/>  <!-- Body length -->
+<xacro:property name="bl" value="0.60"/>   <!-- body length (X) -->
+<xacro:property name="bw" value="0.30"/>   <!-- body width  (Y) -->
+<xacro:property name="bh" value="0.20"/>   <!-- body height (Z) -->
 <!-- LiDAR Dimensions -->
 <xacro:property name="lr" value="0.15"/> <!-- LiDAR Radius -->
 <xacro:property name="ll" value="0.1"/>  <!-- LiDAR Length -->
-<!-- TODO: Set Distances -->
-<!-- Distances Between Certain Centres -->
-<xacro:property name="s1" value="${b/2 + r}"/>
-<xacro:property name="s2" value="${r*2}"/>
-<xacro:property name="s3" value="${r*2}"/>
-<xacro:property name="s4" value="${c/2 + d/2}"/>
+<!-- ################################################    -->
+<!--            Location Setup                           -->
+<!--            MARK: LOCO                               -->
+<!-- ################################################    -->
+<!-- Arm / pivot geometry -->
+<xacro:property name="pivot_margin" value="0.02"/>  <!-- keep pivot inside body end -->
+<xacro:property name="xp" value="0.10"/>            <!-- track COM -> pivot along +X -->
+<!-- Pivot locations on the body (X axis) -->
+<xacro:property name="pivot_x_front" value="${ bl/2 - pivot_margin }"/>
+<xacro:property name="pivot_x_rear"  value="${-(bl/2 - pivot_margin)}"/>
+<!-- Track COM X positions (because track link origin is COM) -->
+<xacro:property name="track_com_x_front" value="${ pivot_x_front - xp }"/>
+<xacro:property name="track_com_x_rear"  value="${ pivot_x_rear  - xp }"/>
+<!-- Left/right track COM Y placement -->
+<xacro:property name="track_com_y" value="${ bw/2 + tw/2 }"/>
+<!-- Body Z placement above ground (simple + stable version) -->
+<xacro:property name="body_z_from_ground" value="${ th/2 + bh/2 }"/>
 <!-- ################################################    -->
 <!--                  Mass & Inertia                     -->
@@ -62,12 +72,12 @@
 <!-- ################################################    -->
 <!-- Densities -->
-<xacro:property name="body_desnity" value="2710.0"/>  <!-- body -->
-<xacro:property name="track_desnity" value="2710.0"/>  <!-- track -->\
+<xacro:property name="body_density" value="2710.0"/>  <!-- body -->
+<xacro:property name="track_density" value="2710.0"/>  <!-- track -->\
  <!-- LiDAR density is not set as it would affect the spin of
  the LiDAR if we were to set it. That being said the spin is
  not simulated so we do not need to worry about it.-->
 <!-- Masses -->
-<xacro:property name="body_mass" value="${body_desnity*bl*bh*bw}"/>
-<xacro:property name="track_mass" value="${track_desnity*tl*th*tw}"/>
+<xacro:property name="body_mass" value="${body_density*bl*bh*bw}"/>
+<xacro:property name="track_mass" value="${track_density*tl*th*tw}"/>
 <!-- Body inertia -->
 <xacro:property name="Ix_body" value="${(1.0/12.0)*body_mass*(bh*bh + bw*bw)}"/>
@@ -79,9 +89,21 @@
 <xacro:property name="Iz_track" value="${(1.0/12.0)*mT*(tl*tl + tw*tw)}"/>
 <!-- Inertia macros -->
+<xacro:macro name="inertia_body">
+    <inertial>
+        <mass value="${body_mass}"/>
+        <inertia ixx="${Ix_body}" ixy="0" ixz="0" iyy="${Iy_body}" iyz="0" izz="${Iz_body}"/>
+    </inertial>
+</xacro:macro>
+<xacro:macro name="inertia_track">
+    <inertial>
+        <mass value="${track_mass}"/>
+        <inertia ixx="${Ix_track}" ixy="0" ixz="0" iyy="${Iy_track}" iyz="0" izz="${Iz_track}"/>
+    </inertial>
+</xacro:macro>
 <!-- ################################################ -->
 <!--            Include Additional Files              -->
 <!--            MARK: File Incl.                      -->
 <!-- ################################################ -->
-<!-- <xacro:include filename="$(find ember_robot)/model/robot.gazebo"/> -->
+<xacro:include filename="$(find ember_robot)/model/ember.gazebo"/>
 <!-- ################################################ -->
 <!-- MARK: LINKS, JOINTS HERE                        -->
@@ -90,4 +112,9 @@
 <!-- START: Fictitious Link of the Robot              -->
 <!-- ################################################ -->
+<link name="base_footprint"/>
+<joint name="body_link_joint" type="fixed">
+    <parent link="base_footprint"/>
+    <child link="body_link"/>
+</joint>
 <!-- ################################################ -->
 <!-- END: Fictitious Link of the Robot                -->
@@ -96,4 +123,19 @@
 <!-- START: Body Link of the Robot                    -->
 <!-- ################################################ -->
+<link name="body_link">
+    <visual>
+        <geometry>
+            <box size="${bl} ${bh} ${bw}"/>
+        </geometry>
+        <origin rpy="0 0 0" xyz="0 0 ${s1}"/>
+    </visual>
+    <collision>
+        <geometry>
+            <box size="${bl} ${bh} ${bw}"/>
+        </geometry>
+        <origin rpy="0 0 0" xyz="0 0 ${body_z_from_ground}"/>
+    </collision>
+    <xacro:inertia_body/>
+</link>
 <!-- ################################################ -->
 <!-- END: Body Link of the Robot                      -->
@@ -135,4 +177,3 @@
 <!-- END: LiDAR                                         -->
 <!-- ################################################  -->
-<!-- TODO: When completed  -->
-<!-- </robot> -->
+</robot>

Commit message: robot exists :)

File: LiDAR_Simulation/heatsim_ws/src/ember_robot/model/ember.xacro (robot description, xacro)
@@ -11,4 +11,10 @@
 -->
 <!-- ################################################    -->
+<!--
+Orientation:
+    x -> Forward
+    y -> Left
+    z -> Up
+-->
 <!-- Robot Part Names:
 Tracks:
@@ -85,7 +91,7 @@
 <xacro:property name="Iz_body" value="${(1.0/12.0)*body_mass*(bl*bl + bw*bw)}"/>
 <!-- Track inertia -->
-<xacro:property name="Ix_track" value="${(1.0/12.0)*mT*(tw*tw + th*th)}"/>
-<xacro:property name="Iy_track" value="${(1.0/12.0)*mT*(tl*tl + th*th)}"/>
-<xacro:property name="Iz_track" value="${(1.0/12.0)*mT*(tl*tl + tw*tw)}"/>
+<xacro:property name="Ix_track" value="${(1.0/12.0)*track_mass*(tw*tw + th*th)}"/>
+<xacro:property name="Iy_track" value="${(1.0/12.0)*track_mass*(tl*tl + th*th)}"/>
+<xacro:property name="Iz_track" value="${(1.0/12.0)*track_mass*(tl*tl + tw*tw)}"/>
 <!-- Inertia macros -->
 <xacro:macro name="inertia_body">
@@ -128,5 +134,5 @@
             <box size="${bl} ${bh} ${bw}"/>
         </geometry>
-        <origin rpy="0 0 0" xyz="0 0 ${s1}"/>
+        <origin rpy="0 0 0" xyz="0 0 ${body_z_from_ground}"/>
     </visual>
     <collision>
@@ -144,4 +150,21 @@
 <!-- START: Front Left Track of the Robot + Joint      -->
 <!-- ################################################  -->
+<joint name="front_left_track_joint" type="continuous">
+    <parent link="body_link"/>
+    <child link="flt_link"/>
+    <origin xyz="${pivot_x_front} ${track_com_y} ${tw}" rpy="0 0 0"/>
+    <axis xyz="0 1 0"/>
+</joint>
+<link name="flt_link">
+    <visual>
+        <origin xyz="${-xp} 0 0" rpy="0 0 0"/>
+        <geometry><box size="${tl} ${tw} ${th}"/></geometry>
+    </visual>
+    <collision>
+        <origin xyz="${-xp} 0 0" rpy="0 0 0"/>
+        <geometry><box size="${tl} ${tw} ${th}"/></geometry>
+    </collision>
+    <xacro:inertia_track/>
+</link>
 <!-- ################################################  -->
 <!-- END: Front Left Track                             -->
@@ -150,4 +173,21 @@
 <!-- START: Front Right Track of the Robot + Joint     -->
 <!-- ################################################  -->
+<joint name="front_right_track_joint" type="continuous">
+    <parent link="body_link"/>
+    <child link="frt_link"/>
+    <origin xyz="${pivot_x_front} ${-track_com_y} ${tw}" rpy="0 0 0"/>
+    <axis xyz="0 1 0"/>
+</joint>
+<link name="frt_link">
+    <visual>
+        <origin xyz="${-xp} 0 0" rpy="0 0 0"/>
+        <geometry><box size="${tl} ${tw} ${th}"/></geometry>
+    </visual>
+    <collision>
+        <origin xyz="${-xp} 0 0" rpy="0 0 0"/>
+        <geometry><box size="${tl} ${tw} ${th}"/></geometry>
+    </collision>
+    <xacro:inertia_track/>
+</link>
 <!-- ################################################  -->
 <!-- END: Front Right Track                            -->
@@ -156,4 +196,21 @@
 <!-- START: Back Left Track of the Robot + Joint       -->
 <!-- ################################################  -->
+<joint name="back_left_track_joint" type="continuous">
+    <parent link="body_link"/>
+    <child link="blt_link"/>
+    <origin xyz="${-pivot_x_front} ${track_com_y} ${tw}" rpy="0 0 0"/>
+    <axis xyz="0 1 0"/>
+</joint>
+<link name="blt_link">
+    <visual>
+        <origin xyz="${xp} 0 0" rpy="0 0 0"/>
+        <geometry><box size="${tl} ${tw} ${th}"/></geometry>
+    </visual>
+    <collision>
+        <origin xyz="${xp} 0 0" rpy="0 0 0"/>
+        <geometry><box size="${tl} ${tw} ${th}"/></geometry>
+    </collision>
+    <xacro:inertia_track/>
+</link>
 <!-- ################################################  -->
 <!-- END: Back Left Track                              -->
@@ -162,16 +219,47 @@
 <!-- START: Back Right Track of the Robot + Joint       -->
 <!-- ################################################  -->
+<joint name="back_right_track_joint" type="continuous">
+    <parent link="body_link"/>
+    <child link="brt_link"/>
+    <origin xyz="${-pivot_x_front} ${-track_com_y} ${tw}" rpy="0 0 0"/>
+    <axis xyz="0 1 0"/>
+</joint>
+<link name="brt_link">
+    <visual>
+        <origin xyz="${xp} 0 0" rpy="0 0 0"/>
+        <geometry><box size="${tl} ${tw} ${th}"/></geometry>
+    </visual>
+    <collision>
+        <origin xyz="${xp} 0 0" rpy="0 0 0"/>
+        <geometry><box size="${tl} ${tw} ${th}"/></geometry>
+    </collision>
+    <xacro:inertia_track/>
+</link>
 <!-- ################################################  -->
 <!-- END: Back Right Track                              -->
 <!-- ################################################  -->
 <!-- ################################################  -->
-<!-- START:Tank Track                                -->
-<!-- ################################################  -->
-<!-- ################################################  -->
-<!-- END:Tank Track                                  -->
-<!-- ################################################  -->
-<!-- ################################################  -->
 <!-- START: LiDAR                                       -->
 <!-- ################################################  -->
+<joint name="lidar_joint" type="fixed">
+    <parent link="body_link"/>
+    <child link="lidar_link"/>
+    <origin xyz="0.0 0 0.5" rpy="0 0 0"/>
+</joint>
+<link name="lidar_link">
+    <visual>
+        <origin xyz="0 0 0" rpy="0 0 0"/>
+        <geometry><cylinder radius="0.1" length="0.1"/></geometry>
+    </visual>
+    <collision>
+        <origin xyz="0 0 0" rpy="0 0 0"/>
+        <geometry><cylinder radius="0.1" length="0.1"/></geometry>
+    </collision>
+    <!-- Minimal but valid inertia -->
+    <inertial>
+        <mass value="1e-6"/>
+        <inertia ixx="1e-6" ixy="0" ixz="0" iyy="1e-6" iyz="0" izz="1e-6"/>
+    </inertial>
+</link>
 <!-- ################################################  -->
 <!-- END: LiDAR                                         -->
