Commit message: LiDAR made

File: LiDAR_Simulation/heatsim_ws/src/ember_robot/3D_LiDAR/SF45B_LiDAR.xacro (robot description, xacro)
@@ -1,123 +1,106 @@
 <?xml version="1.0"?>
-<robot name="ember_bot" xmlns:xacro="http://www.ros.org/wiki/xacro">
-<!-- ################################################    -->
-<!--            Geometry & Constants                     -->
-<!-- ################################################    -->
-<xacro:property name="lr" value="0.1"/>   <!-- LiDAR Radius -->
-<xacro:property name="ll" value="0.1"/>   <!-- LiDAR Length -->
-<xacro:property name="body_length" value="0.6"/>
-<xacro:property name="body_width" value="0.4"/>
-<xacro:property name="body_height" value="0.2"/>
-<!-- ################################################ -->
-<!--            Include Additional Files              -->
-<!-- ################################################ -->
-<xacro:include filename="$(find ember_robot)/3D_LiDAR/SF45B_LiDAR.gazebo"/>
-<!-- ################################################ -->
-<!-- Fictitious Base Link                             -->
-<!-- ################################################ -->
-<link name="base_footprint"/>
-<!-- ################################################ -->
-<!-- Body Link                                        -->
-<!-- ################################################ -->
-<link name="body_link">
-    <visual>
-        <origin xyz="0 0 0" rpy="0 0 0"/>
-        <geometry>
-            <box size="${body_length} ${body_width} ${body_height}"/>
-        </geometry>
-        <material name="gray">
-            <color rgba="0.5 0.5 0.5 1.0"/>
-        </material>
+<robot name="SF45B_lidar">
+  <!-- BASE LINK (Cylindar) -->
+  <link name="base">
+    <inertial>
+      <origin xyz="0 0 0.029335" rpy="0 0 0"/>
+      <mass value="1.2"/>
+      <inertia ixx="0.001087473" ixy="0" ixz="0"
+               iyy="0.001087473" iyz="0"
+               izz="0.001092437"/>
+    </inertial>
+    <collision name="base_collision">
+      <origin xyz="0 0 0.029335" rpy="0 0 0"/>
+      <geometry>
+        <cylinder radius="0.04267" length="0.05867"/>
+      </geometry>
+    </collision>
+    <visual name="base_visual">
+      <origin xyz="0 0 0.029335" rpy="0 0 0"/>
+      <geometry>
+        <cylinder radius="0.04267" length="0.05867"/>
+      </geometry>
+      <material name="Blue">
+        <color rgba="0.1 0.3 0.9 1"/>
+      </material>
     </visual>
-    <collision>
-        <origin xyz="0 0 0" rpy="0 0 0"/>
-        <geometry>
-            <box size="${body_length} ${body_width} ${body_height}"/>
-        </geometry>
+  </link>
+  <!-- TOP LINK (Cylindar) -->
+  <!-- Enable Sensors Engine (Ignition/Gazebo Sim) -->
+  <link name="top">
+    <inertial>
+      <origin xyz="0 0 0" rpy="0 0 0"/>
+      <mass value="0.1"/>
+      <inertia ixx="0.000090623" ixy="0" ixz="0"
+               iyy="0.000090623" iyz="0"
+               izz="0.000091036"/>
+    </inertial>
+    <collision name="top_collision">
+      <origin xyz="0 0 0" rpy="0 0 0"/>
+      <geometry>
+        <cylinder radius="0.04267" length="0.05867"/>
+      </geometry>
     </collision>
-    <inertial>
-        <mass value="5.0"/>
-        <origin xyz="0 0 0" rpy="0 0 0"/>
-        <inertia
-            ixx="0.1" ixy="0.0" ixz="0.0"
-            iyy="0.1" iyz="0.0"
-            izz="0.1"/>
-    </inertial>
-</link>
-<joint name="body_link_joint" type="fixed">
-    <parent link="base_footprint"/>
-    <child link="body_link"/>
-    <origin xyz="0 0 ${body_height/2}" rpy="0 0 0"/>
-</joint>
-<!-- ################################################ -->
-<!-- LiDAR Base Link                                  -->
-<!-- ################################################ -->
-<link name="lidar_base_link">
-    <visual>
-        <origin xyz="0 0 0" rpy="0 0 0"/>
-        <geometry>
-            <cylinder radius="${lr}" length="${ll}"/>
-        </geometry>
-        <material name="dark_gray">
-            <color rgba="0.3 0.3 0.3 1.0"/>
-        </material>
+    <visual name="top_visual">
+      <origin xyz="0 0 0" rpy="0 0 0"/>
+      <geometry>
+        <cylinder radius="0.04267" length="0.05867"/>
+      </geometry>
+      <material name="DarkGray">
+        <color rgba="0.25 0.25 0.25 1"/>
+      </material>
     </visual>
-    <collision>
-        <origin xyz="0 0 0" rpy="0 0 0"/>
-        <geometry>
-            <cylinder radius="${lr}" length="${ll}"/>
-        </geometry>
-    </collision>
-    <inertial>
-        <mass value="0.5"/>
-        <origin xyz="0 0 0" rpy="0 0 0"/>
-        <inertia
-            ixx="0.001" ixy="0" ixz="0"
-            iyy="0.001" iyz="0"
-            izz="0.001"/>
-    </inertial>
-</link>
-<!-- Connect LiDAR base to body -->
-<joint name="lidar_base_joint" type="fixed">
-    <parent link="body_link"/>
-    <child link="lidar_base__link"/>
-    <origin xyz="${body_length/2 - 0.05} 0 ${body_height/2 + ll/2}" rpy="0 0 0"/>
-</joint>
-<!-- ################################################ -->
-<!-- LiDAR Sensor Link                                -->
-<!-- ################################################ -->
-<link name="lidar_link">
-    <visual>
-        <origin xyz="0 0 0" rpy="0 0 0"/>
-        <geometry>
-            <cylinder radius="${lr}" length="${ll}"/>
-        </geometry>
-        <material name="blue">
-            <color rgba="0.0 0.0 1.0 1.0"/>
-        </material>
-    </visual>
-    <collision>
-        <origin xyz="0 0 0" rpy="0 0 0"/>
-        <geometry>
-            <cylinder radius="${lr}" length="${ll}"/>
-        </geometry>
-    </collision>
-    <inertial>
-        <mass value="0.3"/>
-        <origin xyz="0 0 0" rpy="0 0 0"/>
-        <inertia
-            ixx="0.001" ixy="0" ixz="0"
-            iyy="0.001" iyz="0"
-            izz="0.001"/>
-    </inertial>
-</link>
-<!-- LiDAR rotating joint -->
-<joint name="lidar_joint" type="revolute">
-    <parent link="lidar_base__link"/>
-    <child link="lidar_link"/>
-    <origin xyz="0.0 0 ${ll/2}" rpy="0 0 0"/>
+  </link>
+  <!-- REVOLUTE JOINT (Continuous Spin) -->
+  <joint name="joint" type="continuous">
+    <origin xyz="0 0 0.088005" rpy="0 0 0"/>
+    <parent link="base"/>
+    <child link="top"/>
     <axis xyz="0 0 1"/>
-    <limit lower="-3.14159" upper="3.14159" effort="10" velocity="1.0"/>
-    <dynamics damping="0.1" friction="0.1"/>
-</joint>
+    <limit effort="10" velocity="6.28"/>
+  </joint>
+  <!-- Gazebo Sim GPU LiDAR Sensor (attached to "top") -->
+  <gazebo>
+    <plugin filename="gz-sim-sensors-system" name="gz::sim::systems::Sensors">
+        <render_engine>ogre2</render_engine>
+    </plugin>
+  </gazebo>
+  <gazebo reference="top">
+    <sensor name="gpu_lidar_sensor" type="gpu_lidar">
+      <pose relative_to="top">0 0 0 0 0 0</pose>
+      <visualize>1</visualize>
+      <always_on>1</always_on>
+      <update_rate>10</update_rate>
+      <!-- gz transport topic -->
+      <topic>scan</topic>
+      <lidar>
+        <scan>
+          <horizontal>
+            <!-- 360 deg sweep -->
+            <samples>720</samples>
+            <resolution>1</resolution>
+            <min_angle>-3.14159265359</min_angle>
+            <max_angle> 3.14159265359</max_angle>
+          </horizontal>
+          <vertical>
+            <!-- 32 channels (HDL-32-ish), using YOUR vertical FOV numbers -->
+            <samples>32</samples>
+            <resolution>1</resolution>
+            <min_angle>-0.53529248</min_angle>
+            <max_angle> 0.18622663</max_angle>
+          </vertical>
+        </scan>
+        <range>
+          <min>0.05</min>
+          <max>70</max>
+          <resolution>0.02</resolution>
+        </range>
+        <noise>
+          <type>gaussian</type>
+          <mean>0.0</mean>
+          <stddev>0.01</stddev>
+        </noise>
+      </lidar>
+    </sensor>
+  </gazebo>
 </robot>
