Commit message: Got Thermal Camera Visual to show, sensor and tf are still not linking properly

File: LiDAR_Simulation/heatsim_ws/src/ember_robot/ember_model/urdf/sensors/FLIR_Lepton_ThermalCamera/FLIR_Lepton.xacro (robot description, xacro)
@@ -15,7 +15,5 @@
       <collision name="base_collision">
         <geometry>
-          <box>
-            <size>${panel_t} ${panel_w} ${panel_h}</size>
-          </box>
+          <box size="${panel_t} ${panel_w} ${panel_h}"/>
         </geometry>
       </collision>
@@ -23,7 +21,5 @@
       <visual name="thermal_visual">
         <geometry>
-          <box>
-            <size>${panel_t} ${panel_w} ${panel_h}</size>
-          </box>
+          <box size="${panel_t} ${panel_w} ${panel_h}"/>
         </geometry>
         <material name="Thermal_Orange">
@@ -59,5 +55,5 @@
   </xacro:macro>
   <!-- Panel dimensions -->
-  <xacro:property name="panel_t" value="0.10"/>   <!-- thickness (x) -->
+  <xacro:property name="panel_t" value="0.02"/>   <!-- thickness (x) -->
   <xacro:property name="panel_w" value="0.18"/>   <!-- width (y) -->
   <xacro:property name="panel_h" value="0.12"/>   <!-- height (z) -->
